File: tlbox/apps/sbr/pcb_v1/pwm_controller.kicad_sch (KiCad schematic)
At the start: 1 part, among them J1 Conn_01x06_Pin

Commit message: Schematic modifications
Connections:
- net VCC: now reaches J1.5 (Pin_5)
- net GND: now reaches J1.6 (Pin_6)
- no-connect marks 4 -> 2
Other:
- note added: "Even though they say the lower voltage limit is 4.8 volts, I have successfully operated it off of 3.3 volts, though obviously there's no guarantee of reliable, flawless behavior beyond the official specs."
- note added: "https://hobbyking.com/en_us/hobby-king-2-4ghz-receiver-6ch-v2.html"
Changed lines of the file:
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@@
 	(generator_version "10.0")
 	(paper "A4")
+	(text "https://hobbyking.com/en_us/hobby-king-2-4ghz-receiver-6ch-v2.html"
+		(exclude_from_sim no)
+		(at 111.506 42.418 0)
+		(effects
+			(font
+				(size 1.27 1.27)
+			)
+		)
+	)
+	(text "Even though they say the lower voltage limit is 4.8 volts, I have successfully operated it off of 3.3 volts, though obviously there's no\nguarantee of reliable, flawless behavior beyond the official specs. "
+		(exclude_from_sim no)
+		(at 113.792 84.582 0)
+		(effects
+			(font
+				(size 1.27 1.27)
+			)
+		)
+	)
 	(text_box "TODO: How to add these external modules best here?"
 		(exclude_from_sim no)
@@
 	)
 	(no_connect
-		(at 111.76 73.66)
+		(at 111.76 60.96)
 	)
-	(no_connect
-		(at 111.76 71.12)
-	)
-	(no_connect
-		(at 111.76 60.96)
+	(hierarchical_label "GND"
+		(shape input)
+		(at 111.76 73.66 0)
+		(effects
+			(font
+				(size 1.27 1.27)
+			)
+			(justify left)
+		)
 	)
 	(hierarchical_label "pwm_throttle"
@@
 		(effects
 			(font
+				(size 1.27 1.27)
+			)
+			(justify left)
+		)
+	)
+	(hierarchical_label "VCC"
+		(shape input)
+		(at 111.76 71.12 0)
+		(effects
+			(font
