File: tlbox/apps/sbr/pcb_v1/self_balancing_robot_v1.kicad_sch (KiCad schematic)
At the start: 0 parts

Commit message: content hashing
Other:
- sheet pwm_controller ports: added GND, VCC; removed none
- sheet uart_radio ports: added GND, VCC; removed none
- note added: "don't we want this pulled up?"
Changed lines of the file:
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@@
 	(generator_version "10.0")
 	(paper "A4")
+	(text "don't we want this pulled up?"
+		(exclude_from_sim no)
+		(at 136.144 111.252 0)
+		(effects
+			(font
+				(size 1.27 1.27)
+			)
+		)
+	)
 	(junction
 		(at 83.82 58.42)
@@
 	)
 	(junction
+		(at 83.82 86.36)
+		(diameter 0)
+		(color 0 0 0 0)
+	)
+	(junction
+		(at 154.94 58.42)
+		(diameter 0)
+		(color 0 0 0 0)
+	)
+	(junction
 		(at 83.82 95.25)
 		(diameter 0)
@@
 	)
 	(junction
+		(at 161.29 58.42)
+		(diameter 0)
+		(color 0 0 0 0)
+	)
+	(junction
 		(at 86.36 55.88)
+		(diameter 0)
+		(color 0 0 0 0)
+	)
+	(junction
+		(at 83.82 64.77)
 		(diameter 0)
 		(color 0 0 0 0)
@@
 	(wire
 		(pts
+			(xy 83.82 64.77) (xy 83.82 74.93)
+		)
+		(stroke
+			(width 0)
+			(type default)
+		)
+	)
+	(wire
+		(pts
+			(xy 162.56 80.01) (xy 154.94 80.01)
+		)
+		(stroke
+			(width 0)
+			(type default)
+		)
+	)
+	(wire
+		(pts
 			(xy 147.32 72.39) (xy 152.4 72.39)
 		)
@@
 	(wire
 		(pts
+			(xy 162.56 64.77) (xy 161.29 64.77)
+		)
+		(stroke
+			(width 0)
+			(type default)
+		)
+	)
+	(wire
+		(pts
+			(xy 154.94 80.01) (xy 154.94 58.42)
+		)
+		(stroke
+			(width 0)
+			(type default)
+		)
+	)
+	(wire
+		(pts
+			(xy 83.82 86.36) (xy 83.82 95.25)
+		)
+		(stroke
+			(width 0)
+			(type default)
+		)
+	)
+	(wire
+		(pts
+			(xy 158.75 67.31) (xy 158.75 64.77)
+		)
+		(stroke
+			(width 0)
+			(type default)
+		)
+	)
+	(wire
+		(pts
 			(xy 209.55 72.39) (xy 152.4 72.39)
 		)
@@
 	(wire
 		(pts
-			(xy 186.69 85.09) (xy 209.55 85.09)
+			(xy 186.69 82.55) (xy 209.55 82.55)
 		)
 		(stroke
@@
 	(wire
 		(pts
-			(xy 186.69 82.55) (xy 209.55 82.55)
-		)
-		(stroke
-			(width 0)
-			(type default)
-		)
-	)
-	(wire
-		(pts
 			(xy 156.21 110.49) (xy 152.4 110.49)
 		)
@@
 	(wire
 		(pts
+			(xy 162.56 67.31) (xy 158.75 67.31)
+		)
+		(stroke
+			(width 0)
+			(type default)
+		)
+	)
+	(wire
+		(pts
+			(xy 154.94 86.36) (xy 83.82 86.36)
+		)
+		(stroke
+			(width 0)
+			(type default)
+		)
+	)
+	(wire
+		(pts
 			(xy 151.13 74.93) (xy 151.13 106.68)
 		)
@@
 	(wire
 		(pts
+			(xy 162.56 82.55) (xy 154.94 82.55)
+		)
+		(stroke
+			(width 0)
+			(type default)
+		)
+	)
+	(wire
+		(pts
 			(xy 113.03 58.42) (xy 113.03 72.39)
 		)
@@
 	(wire
 		(pts
-			(xy 83.82 74.93) (xy 83.82 95.25)
+			(xy 83.82 74.93) (xy 83.82 86.36)
 		)
 		(stroke
@@
 	(wire
 		(pts
+			(xy 154.94 58.42) (xy 113.03 58.42)
+		)
+		(stroke
+			(width 0)
+			(type default)
+		)
+	)
+	(wire
+		(pts
 			(xy 186.69 99.06) (xy 209.55 99.06)
 		)
@@
 	(wire
 		(pts
+			(xy 83.82 64.77) (xy 158.75 64.77)
+		)
+		(stroke
+			(width 0)
+			(type default)
+		)
+	)
+	(wire
+		(pts
+			(xy 186.69 80.01) (xy 209.55 80.01)
+		)
+		(stroke
+			(width 0)
+			(type default)
+		)
+	)
+	(wire
+		(pts
+			(xy 161.29 64.77) (xy 161.29 58.42)
+		)
+		(stroke
+			(width 0)
+			(type default)
+		)
+	)
+	(wire
+		(pts
 			(xy 152.4 72.39) (xy 152.4 104.14)
 		)
@@
 	(wire
 		(pts
-			(xy 209.55 58.42) (xy 113.03 58.42)
+			(xy 209.55 58.42) (xy 161.29 58.42)
 		)
 		(stroke
@@
 	(wire
 		(pts
-			(xy 83.82 58.42) (xy 83.82 74.93)
+			(xy 83.82 58.42) (xy 83.82 64.77)
 		)
 		(stroke
@@
 	(wire
 		(pts
+			(xy 161.29 58.42) (xy 154.94 58.42)
+		)
+		(stroke
+			(width 0)
+			(type default)
+		)
+	)
+	(wire
+		(pts
 			(xy 113.03 72.39) (xy 116.84 72.39)
 		)
@@
 		(pts
 			(xy 111.76 55.88) (xy 209.55 55.88)
+		)
+		(stroke
+			(width 0)
+			(type default)
+		)
+	)
+	(wire
+		(pts
+			(xy 154.94 82.55) (xy 154.94 86.36)
 		)
 		(stroke
@@
 		)
 		(pin "uart_from_micro" output
-			(at 209.55 85.09 180)
+			(at 209.55 82.55 180)
 			(effects
 				(font
@@
 		)
 		(pin "uart_to_micro" input
-			(at 209.55 82.55 180)
+			(at 209.55 80.01 180)
 			(effects
 				(font
@@
 	)
 	(sheet
-		(at 168.91 80.01)
-		(size 17.78 7.62)
+		(at 162.56 77.47)
+		(size 24.13 7.62)
 		(exclude_from_sim no)
 		(in_bom yes)
@@
 		)
 		(property "Sheetname" "uart_radio"
-			(at 168.91 79.2984 0)
+			(at 162.56 76.7584 0)
 			(show_name no)
 			(do_not_autoplace no)
@@
 		)
 		(property "Sheetfile" "uart_radio.kicad_sch"
-			(at 168.91 88.2146 0)
+			(at 162.56 85.6746 0)
 			(hide yes)
 			(show_name no)
@@
 		)
 		(pin "uart_from_radio" output
+			(at 186.69 80.01 0)
+			(effects
+				(font
+					(size 1.27 1.27)
+				)
+				(justify right)
+			)
+		)
+		(pin "uart_to_radio" input
 			(at 186.69 82.55 0)
 			(effects
@@
 			)
 		)
-		(pin "uart_to_radio" input
-			(at 186.69 85.09 0)
-			(effects
-				(font
-					(size 1.27 1.27)
-				)
-				(justify right)
+		(pin "GND" input
+			(at 162.56 82.55 180)
+			(effects
+				(font
+					(size 1.27 1.27)
+				)
+				(justify left)
+			)
+		)
+		(pin "VCC" input
+			(at 162.56 80.01 180)
+			(effects
+				(font
+					(size 1.27 1.27)
+				)
+				(justify left)
 			)
 		)
@@
 	)
 	(sheet
-		(at 171.45 62.23)
-		(size 15.24 7.62)
+		(at 162.56 62.23)
+		(size 24.13 7.62)
 		(exclude_from_sim no)
 		(in_bom yes)
@@
 		)
 		(property "Sheetname" "pwm_controller"
-			(at 171.45 61.5184 0)
+			(at 162.56 61.5184 0)
 			(show_name no)
 			(do_not_autoplace no)
@@
 		)
 		(property "Sheetfile" "pwm_controller.kicad_sch"
-			(at 171.45 70.4346 0)
+			(at 162.56 70.4346 0)
 			(hide yes)
 			(show_name no)
@@
 			)
 		)
+		(pin "GND" input
+			(at 162.56 67.31 180)
+			(effects
+				(font
+					(size 1.27 1.27)
+				)
+				(justify left)
+			)
+		)
+		(pin "VCC" input
+			(at 162.56 64.77 180)
+			(effects
+				(font
+					(size 1.27 1.27)
+				)
+				(justify left)
+			)
+		)
