File: tlbox/apps/sbr/pcb_v1/uart_radio.kicad_sch (KiCad schematic)
At the start: 1 part, among them J2 Conn_01x02_Pin

Commit message: content hashing
Parts:
- removed J2: Conn_01x02_Pin, symbol Connector:Conn_01x02_Pin
- added J4: Conn_01x04_Pin, symbol Connector:Conn_01x04_Pin
Connections:
- net uart_from_radio: now also J4.1 (Pin_1)
- net uart_to_radio: now also J4.2 (Pin_2)
- new net GND: J4.4 (Pin_4)
- new net VCC: J4.3 (Pin_3)
Other:
- note added: "Labeled as 5V"
Changed lines of the file:
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@@
 	(generator_version "10.0")
 	(paper "A4")
+	(text "Labeled as 5V"
+		(exclude_from_sim no)
+		(at 139.954 78.994 0)
+		(effects
+			(font
+				(size 1.27 1.27)
+			)
+		)
+	)
+	(wire
+		(pts
+			(xy 115.57 78.74) (xy 119.38 78.74)
+		)
+		(stroke
+			(width 0)
+			(type default)
+		)
+	)
+	(wire
+		(pts
+			(xy 115.57 81.28) (xy 119.38 81.28)
+		)
+		(stroke
+			(width 0)
+			(type default)
+		)
+	)
+	(wire
+		(pts
+			(xy 119.38 73.66) (xy 115.57 73.66)
+		)
+		(stroke
+			(width 0)
+			(type default)
+		)
+	)
+	(wire
+		(pts
+			(xy 119.38 76.2) (xy 115.57 76.2)
+		)
+		(stroke
+			(width 0)
+			(type default)
+		)
+	)
 	(hierarchical_label "uart_from_radio"
 		(shape output)
-		(at 115.57 62.23 0)
+		(at 119.38 73.66 0)
 		(effects
 			(font
@@
 	(hierarchical_label "uart_to_radio"
 		(shape input)
-		(at 115.57 64.77 0)
+		(at 119.38 76.2 0)
+		(effects
+			(font
+				(size 1.27 1.27)
+			)
+			(justify left)
+		)
+	)
+	(hierarchical_label "VCC"
+		(shape input)
+		(at 119.38 78.74 0)
+		(effects
+			(font
+				(size 1.27 1.27)
+			)
+			(justify left)
+		)
+	)
+	(hierarchical_label "GND"
+		(shape input)
+		(at 119.38 81.28 0)
 		(effects
 			(font
@@
 	)
 	(symbol
-		(lib_id "Connector:Conn_01x02_Pin")
-		(at 110.49 62.23 0)
+		(lib_id "Connector:Conn_01x04_Pin")
+		(at 110.49 76.2 0)
 		(unit 1)
 		(body_style 1)
@@
 		(in_pos_files yes)
 		(dnp no)
-		(property "Reference" "J2"
-			(at 111.125 57.15 0)
+		(fields_autoplaced yes)
+		(property "Reference" "J4"
+			(at 111.125 68.58 0)
 			(show_name no)
 			(do_not_autoplace no)
@@
 			)
 		)
-		(property "Value" "Conn_01x02_Pin"
-			(at 111.125 59.69 0)
+		(property "Value" "Conn_01x04_Pin"
+			(at 111.125 71.12 0)
 			(show_name no)
 			(do_not_autoplace no)
@@
 		)
 		(property "Footprint" ""
-			(at 110.49 62.23 0)
+			(at 110.49 76.2 0)
 			(hide yes)
 			(show_name no)
@@
 		)
 		(property "Datasheet" ""
-			(at 110.49 62.23 0)
+			(at 110.49 76.2 0)
 			(hide yes)
 			(show_name no)
@@
 			)
 		)
-		(property "Description" "Generic connector, single row, 01x02, script generated"
-			(at 109.728 53.086 0)
+		(property "Description" "Generic connector, single row, 01x04, script generated"
+			(at 110.49 76.2 0)
+			(hide yes)
 			(show_name no)
 			(do_not_autoplace no)
@@
 			)
 		)
+		(pin "4"
+		)
 		(pin "2"
+		)
+		(pin "3"
 		)
 		(pin "1"
@@
 			(project "self_balancing_robot_v1"
 				(path "/f1bc52c2-82b2-44ac-a8ec-1286ff19a550/7849255e-dc2a-45a5-ad4e-6c6d20980213"
-					(reference "J2")
+					(reference "J4")
 					(unit 1)
 				)
